File: kicad/bikecomp/bikecomp.sch (KiCad schematic (older format))
At the start: 8 parts

Commit message: Schematics experiments
Parts:
- added Q?: BSS138, Package_TO_SOT_SMD:SOT-23, symbol Transistor_FET:BSS138
- added R? (x2): 22, symbol Device:R
- added R?: 1.5k, symbol Device:R
- added R? (x2): 10k, symbol Device:R
- added R?: R, symbol Device:R
- added R?: R_PHOTO, symbol Device:R_PHOTO
Connections:
- net 2.8V is gone; now on net VDD: J?.3 (Pin_3)
- net CS: now also U?.25 (PB12)
- net D0: now also U?.10 (PA0)
- net D1: now also U?.11 (PA1)
- net D2: now also U?.12 (PA2)
- net D3: now also U?.13 (PA3)
- net D4: now also U?.14 (PA4)
- net D5: now also U?.15 (PA5)
- net D6: now also U?.16 (PA6)
- net D7: now also U?.17 (PA7)
- net GNDD: now also U?.23 (VSS), U?.35 (VSS), U?.47 (VSS), U?.8 (VSSA), Q?.2 (S)
- net RD: now also U?.27 (PB14)
- net RS: now also U?.22 (PB11)
- net RST: now also U?.21 (PB10)
- net WR: now also U?.28 (PB15)
- net VDD: now reaches U?.2 (VO)
- net VDD: now also U?.1 (VBAT), U?.24 (VDD), U?.36 (VDD), U?.48 (VDD), U?.9 (VDDA), R?.1, R?.1, R?.1
- net at U?.4 (EN): now also U?.2 (PC13); no longer U?.19 (PB1)
- net at R?.1, R?.2: now also U?.18 (PB0); no longer U?.10 (PA0)
- net at Q?.1 (G): now also U?.38 (PA15); no longer U?.18 (PB0)
- net BTN0: now reaches U?.20 (PB2)
- net SCK: now reaches U?.26 (PB13)
- net at U?.29 (PA8): now also Q?.1 (G)
- net TX: now reaches U?.30 (PA9)
- net RX: now reaches U?.31 (PA10)
- net at U?.32 (PA11): now also R?.2
- net at U?.33 (PA12): now also R?.2, R?.2
- net SWDIO: now reaches U?.34 (PA13)
- net SWCLK: now reaches U?.37 (PA14)
- net BTN1: now reaches U?.39 (PB3)
- net BTN2: now reaches U?.40 (PB4)
- net BTN3: now reaches U?.41 (PB5)
- net SCL: now reaches U?.42 (PB6)
- net SCL: now also R?.2
- net SDA: now reaches U?.43 (PB7)
- net SDA: now also R?.2
- net WHEEL: now reaches U?.45 (PB8)
- net PEDAL: now reaches U?.46 (PB9)
- new net: R?.1, R?.2, U?.19 (PB1)
- new net: Q?.3 (D), R?.2
- new net USB_DM: R?.1
- new net USB_DP: R?.1
Other:
- moved on the sheet: BT?, J?, Q?, R?, U?

Commit message: Button handling
Connections:
- net BTN0: no longer names the net of U?.20 (PB2)
Changed lines of the file:
@@
 PEDAL
-Wire Wire Line
-	5800 4100 5000 4100
 Wire Wire Line
 	5800 4200 5000 4200
@@
 Wire Wire Line
 	5800 4400 5000 4400
-Text Label 5000 4100 0    50   ~ 0
-BTN0
 Text Label 5000 4200 0    50   ~ 0
 BTN1

Commit message: Update schematics
Parts:
- added C?: 1.0, symbol Device:C
- added C?: 4.7, symbol Device:CP
- added D?: D_Schottky, symbol Device:D_Schottky
- added L?: 10uH, symbol Device:L
- added R?: 47, symbol Device:R
- U?: value AMS1117-3.3 -> AMS1117-2.5
Connections:
- net GND is gone; now on net GNDD: J?.18 (Pin_18), J?.21 (Pin_21), J?.4 (Pin_4), J?.9 (Pin_9)
- net GNDD: now also U?.2 (GND), C?.2, C?.2, R?.2
- net at BT?.1 (+), R?.1, U?.3 (VI)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: now also C?.1, L?.1
- net LED_N: now reaches U?.3 (FB)
- net LED_N: now also J?.23 (Pin_23), J?.24 (Pin_24), R?.1
- net at Q?.1 (G), U?.38 (PA15): now also Q?.1 (G)
- net at U?.29 (PA8): no longer Q?.1 (G)
- net 10V: no longer names the net of U?.1 (SW)
- net 10V: now also D?.2 (A), L?.2
- net LED renamed LED_P
- net LED_P: now also C?.1, D?.1 (K); no longer J?.23 (Pin_23), J?.24 (Pin_24)
Other:
- moved on the sheet: BT?, U?

Commit message: Update schematic
Parts:
- added C?: 1.0, symbol Device:CP
- added R?: 820k, symbol Device:R
- C?: value 1.0 -> 5.6p
- R?: value 47 -> 150k
- U?: value MT3608 -> TPS61040DBV
Connections:
- net GNDD: now also J?.23 (Pin_23), J?.24 (Pin_24), C?.2; no longer C?.2
- net LED_N: no longer names the net of R?.1, U?.3 (FB)
- net LED_N: now also C?.2, R?.2; no longer J?.23 (Pin_23), J?.24 (Pin_24)
- net LED_P renamed BCKL
- net BCKL: now also C?.1, R?.1
Other:
- moved on the sheet: C?, D?, L?, R?, U?
Changed lines of the file:
@@
 	9250 1850 9550 1850
 Text Label 8400 1650 0    50   ~ 0
-LED_P
+BCKL
 Text Label 8400 1850 0    50   ~ 0
 2.8V
@@
 	2500 2050 2500 2400
 Wire Wire Line
-	6100 1350 6700 1350
+	6350 1350 6700 1350
 Wire Wire Line
 	6700 1350 6700 1850
@@
 L Regulator_Linear:AMS1117-3.3 U?
 U 1 1 5F0BF98F
-P 5800 1350
-F 0 "U?" H 5800 1592 50  0000 C CNN
-F 1 "AMS1117-2.5" H 5800 1501 50  0000 C CNN
-F 2 "Package_TO_SOT_SMD:SOT-223-3_TabPin2" H 5800 1550 50  0001 C CNN
-F 3 "http://www.advanced-monolithic.com/pdf/ds1117.pdf" H 5900 1100 50  0001 C CNN
-	1    5800 1350
+P 6050 1350
+F 0 "U?" H 6050 1592 50  0000 C CNN
+F 1 "AMS1117-2.5" H 6050 1501 50  0000 C CNN
+F 2 "Package_TO_SOT_SMD:SOT-223-3_TabPin2" H 6050 1550 50  0001 C CNN
+F 3 "http://www.advanced-monolithic.com/pdf/ds1117.pdf" H 6150 1100 50  0001 C CNN
+	1    6050 1350
 	1    0    0    -1
 $EndComp
@@
 L power:GNDD #PWR?
 U 1 1 5F0C179F
-P 5800 1950
-F 0 "#PWR?" H 5800 1700 50  0001 C CNN
-F 1 "GNDD" H 5804 1795 50  0000 C CNN
-F 2 "" H 5800 1950 50  0001 C CNN
-F 3 "" H 5800 1950 50  0001 C CNN
-	1    5800 1950
-	1    0    0    -1
-$EndComp
-Wire Wire Line
-	5800 1950 5800 1650
+P 6050 1950
+F 0 "#PWR?" H 6050 1700 50  0001 C CNN
+F 1 "GNDD" H 6054 1795 50  0000 C CNN
+F 2 "" H 6050 1950 50  0001 C CNN
+F 3 "" H 6050 1950 50  0001 C CNN
+	1    6050 1950
+	1    0    0    -1
+$EndComp
+Wire Wire Line
+	6050 1950 6050 1650
 $Comp
 L Device:R R?
@@
 Connection ~ 2500 2050
 Wire Wire Line
-	3400 2250 3250 2250
+	3350 2250 3250 2250
 Wire Wire Line
 	7100 3900 7350 3900
@@
 L Regulator_Switching:MT3608 U?
 U 1 1 5F0C489A
-P 3700 2150
-F 0 "U?" H 3700 2517 50  0000 C CNN
-F 1 "MT3608" H 3700 2426 50  0000 C CNN
-F 2 "Package_TO_SOT_SMD:SOT-23-6" H 3750 1900 50  0001 L CIN
-F 3 "https://www.olimex.com/Products/Breadboarding/BB-PWR-3608/resources/MT3608.pdf" H 3450 2600 50  0001 C CNN
-	1    3700 2150
+P 3650 2150
+F 0 "U?" H 3650 2517 50  0000 C CNN
+F 1 "TPS61040DBV" H 3650 2426 50  0000 C CNN
+F 2 "Package_TO_SOT_SMD:SOT-23-6" H 3700 1900 50  0001 L CIN
+F 3 "https://www.olimex.com/Products/Breadboarding/BB-PWR-3608/resources/MT3608.pdf" H 3400 2600 50  0001 C CNN
+	1    3650 2150
 	1    0    0    -1
 $EndComp
@@
 L power:GNDD #PWR?
 U 1 1 5F20B1E4
-P 3700 2600
-F 0 "#PWR?" H 3700 2350 50  0001 C CNN
-F 1 "GNDD" H 3704 2445 50  0000 C CNN
-F 2 "" H 3700 2600 50  0001 C CNN
-F 3 "" H 3700 2600 50  0001 C CNN
-	1    3700 2600
-	1    0    0    -1
-$EndComp
-Wire Wire Line
-	3700 2600 3700 2450
+P 3650 2600
+F 0 "#PWR?" H 3650 2350 50  0001 C CNN
+F 1 "GNDD" H 3654 2445 50  0000 C CNN
+F 2 "" H 3650 2600 50  0001 C CNN
+F 3 "" H 3650 2600 50  0001 C CNN
+	1    3650 2600
+	1    0    0    -1
+$EndComp
+Wire Wire Line
+	3650 2600 3650 2450
 Wire Wire Line
 	2500 1350 2500 2050
 Wire Wire Line
-	2500 1350 5500 1350
+	2500 1350 5750 1350
 $Comp
 L Device:L L?
 U 1 1 5F225989
-P 3700 1650
-F 0 "L?" V 3890 1650 50  0000 C CNN
-F 1 "10uH" V 3799 1650 50  0000 C CNN
-F 2 "" H 3700 1650 50  0001 C CNN
-F 3 "~" H 3700 1650 50  0001 C CNN
-	1    3700 1650
+P 3650 1650
+F 0 "L?" V 3840 1650 50  0000 C CNN
+F 1 "10uH" V 3749 1650 50  0000 C CNN
+F 2 "" H 3650 1650 50  0001 C CNN
+F 3 "~" H 3650 1650 50  0001 C CNN
+	1    3650 1650
 	0    -1   -1   0
 $EndComp
 Wire Wire Line
-	3850 1650 4100 1650
-Wire Wire Line
-	4100 1650 4100 2050
-Wire Wire Line
-	4100 2050 4000 2050
-Wire Wire Line
-	3550 1650 3250 1650
+	3800 1650 4050 1650
+Wire Wire Line
+	4050 1650 4050 2050
+Wire Wire Line
+	4050 2050 3950 2050
+Wire Wire Line
+	3500 1650 3250 1650
 Wire Wire Line
 	3250 1650 3250 2050
 Connection ~ 3250 2050
 Wire Wire Line
-	3250 2050 3400 2050
+	3250 2050 3350 2050
 $Comp
 L Device:D_Schottky D?
 U 1 1 5F231391
-P 4300 1650
-F 0 "D?" H 4300 1433 50  0000 C CNN
-F 1 "D_Schottky" H 4300 1524 50  0000 C CNN
-F 2 "" H 4300 1650 50  0001 C CNN
-F 3 "~" H 4300 1650 50  0001 C CNN
-	1    4300 1650
+P 4250 1650
+F 0 "D?" H 4250 1433 50  0000 C CNN
+F 1 "D_Schottky" H 4250 1524 50  0000 C CNN
+F 2 "" H 4250 1650 50  0001 C CNN
+F 3 "~" H 4250 1650 50  0001 C CNN
+	1    4250 1650
 	-1   0    0    1
 $EndComp
 Wire Wire Line
-	4150 1650 4100 1650
-Connection ~ 4100 1650
+	4100 1650 4050 1650
+Connection ~ 4050 1650
 $Comp
 L Device:C C?
 U 1 1 5F23C8C5
-P 4550 2000
-F 0 "C?" H 4665 2046 50  0000 L CNN
-F 1 "1.0" H 4665 1955 50  0000 L CNN
-F 2 "" H 4588 1850 50  0001 C CNN
-F 3 "~" H 4550 2000 50  0001 C CNN
-	1    4550 2000
-	1    0    0    -1
-$EndComp
-Wire Wire Line
-	4450 1650 4550 1650
-Wire Wire Line
-	4550 1650 4550 1850
-$Comp
-L power:GNDD #PWR?
-U 1 1 5F2427C0
-P 4550 2300
-F 0 "#PWR?" H 4550 2050 50  0001 C CNN
-F 1 "GNDD" H 4554 2145 50  0000 C CNN
-F 2 "" H 4550 2300 50  0001 C CNN
-F 3 "" H 4550 2300 50  0001 C CNN
-	1    4550 2300
-	1    0    0    -1
-$EndComp
-Wire Wire Line
-	4550 2150 4550 2300
+P 4850 1950
+F 0 "C?" H 4965 1996 50  0000 L CNN
+F 1 "5.6p" H 4965 1905 50  0000 L CNN
+F 2 "" H 4888 1800 50  0001 C CNN
+F 3 "~" H 4850 1950 50  0001 C CNN
+	1    4850 1950
+	1    0    0    -1
+$EndComp
+Wire Wire Line
+	4400 1650 4450 1650
+Wire Wire Line
+	4850 1650 4850 1800
 $Comp
 L Device:CP C?
@@
 	2950 2850 2950 2700
 Wire Wire Line
-	5000 1650 4550 1650
-Connection ~ 4550 1650
+	5500 1650 5200 1650
+Connection ~ 4850 1650
 $Comp
 L Device:R R?
 U 1 1 5F2781F6
-P 4150 2800
-F 0 "R?" H 4220 2846 50  0000 L CNN
-F 1 "47" H 4220 2755 50  0000 L CNN
-F 2 "" V 4080 2800 50  0001 C CNN
-F 3 "~" H 4150 2800 50  0001 C CNN
-	1    4150 2800
+P 4450 2500
+F 0 "R?" H 4520 2546 50  0000 L CNN
+F 1 "150k" H 4520 2455 50  0000 L CNN
+F 2 "" V 4380 2500 50  0001 C CNN
+F 3 "~" H 4450 2500 50  0001 C CNN
+	1    4450 2500
 	1    0    0    -1
 $EndComp
@@
 L power:GNDD #PWR?
 U 1 1 5F27E74F
-P 4150 3050
-F 0 "#PWR?" H 4150 2800 50  0001 C CNN
-F 1 "GNDD" H 4154 2895 50  0000 C CNN
-F 2 "" H 4150 3050 50  0001 C CNN
-F 3 "" H 4150 3050 50  0001 C CNN
-	1    4150 3050
-	1    0    0    -1
-$EndComp
-Wire Wire Line
-	4150 2950 4150 3050
-Wire Wire Line
-	5000 2600 4150 2600
-Wire Wire Line
-	4150 2600 4150 2250
-Wire Wire Line
-	4150 2250 4000 2250
-Wire Wire Line
-	4150 2600 4150 2650
+P 4450 2750
+F 0 "#PWR?" H 4450 2500 50  0001 C CNN
+F 1 "GNDD" H 4454 2595 50  0000 C CNN
+F 2 "" H 4450 2750 50  0001 C CNN
+F 3 "" H 4450 2750 50  0001 C CNN
+	1    4450 2750
+	1    0    0    -1
+$EndComp
+Wire Wire Line
+	4450 2650 4450 2750
+Wire Wire Line
+	4450 2250 3950 2250
 $Comp
 L power:GNDD #PWR?
@@
 Wire Wire Line
 	8650 1650 8750 1650
-Text Label 5000 1650 2    50   ~ 0
-LED_P
-Text Label 5000 2600 2    50   ~ 0
-LED_N
 Wire Wire Line
 	9250 1750 9300 1750
@@
 	9300 1750 9300 1650
 Connection ~ 9300 1650
-Wire Wire Line
-	9300 1650 9700 1650
-Text Label 9700 1650 2    50   ~ 0
-LED_N
 $Comp
 L power:GNDD #PWR?
@@
 	8250 1950 8750 1950
 Connection ~ 8250 2450
-Connection ~ 4150 2600
 Wire Wire Line
 	3050 4500 3050 4750
@@
 Wire Wire Line
 	2050 4500 3050 4500
+$Comp
+L Device:R R?
+U 1 1 5F2D1D8F
+P 4450 1950
+F 0 "R?" H 4520 1996 50  0000 L CNN
+F 1 "820k" H 4520 1905 50  0000 L CNN
+F 2 "" V 4380 1950 50  0001 C CNN
+F 3 "~" H 4450 1950 50  0001 C CNN
+	1    4450 1950
+	1    0    0    -1
+$EndComp
+Wire Wire Line
+	4450 1800 4450 1650
+Connection ~ 4450 1650
+Wire Wire Line
+	4450 1650 4850 1650
+Wire Wire Line
+	4450 2100 4450 2250
+Connection ~ 4450 2250
+Wire Wire Line
+	4450 2250 4450 2350
+Text Label 5500 1650 2    50   ~ 0
+BCKL
+Wire Wire Line
+	9700 1950 9700 1650
+Wire Wire Line
+	9300 1650 9700 1650
+Connection ~ 9700 1950
+Wire Wire Line
+	4450 2250 4850 2250
+Wire Wire Line
+	4850 2100 4850 2250
+$Comp
+L Device:CP C?
+U 1 1 5F2F919A
+P 5200 2450
+F 0 "C?" H 5318 2496 50  0000 L CNN
+F 1 "1.0" H 5318 2405 50  0000 L CNN
+F 2 "" H 5238 2300 50  0001 C CNN
+F 3 "~" H 5200 2450 50  0001 C CNN
+	1    5200 2450
+	1    0    0    -1
+$EndComp
+Wire Wire Line
+	5200 2300 5200 1650
+Connection ~ 5200 1650
+Wire Wire Line
+	5200 1650 4850 1650
+$Comp
+L power:GNDD #PWR?
+U 1 1 5F313A56
+P 5200 2750
+F 0 "#PWR?" H 5200 2500 50  0001 C CNN
+F 1 "GNDD" H 5204 2595 50  0000 C CNN
+F 2 "" H 5200 2750 50  0001 C CNN
+F 3 "" H 5200 2750 50  0001 C CNN
+	1    5200 2750
+	1    0    0    -1
+$EndComp
+Wire Wire Line
+	5200 2750 5200 2600
 $EndSCHEMATC
